Commit message: fix urdf

File: src/imeta_y1_controller/urdf/y1.urdf (robot description, URDF)
Before this commit: robot y1, 8 links, 7 joints
Links:
- link J1_Link: mass 0.34057 -> 0.631
- link J2_Link: mass 0.94239 -> 1.209
- link J3_Link: mass 0.69617 -> 0.916
- link J4_Link: mass 0.27357 -> 0.483
- link J5_Link: mass 0.16994 -> 0.378
- link J6_Link: mass 0.8 -> 0.0001
- link base_link: mass 1.297 -> 1.55068784468738
Joints:
- joint J1_JOINT: limit lower=-2.79 upper=2.79 effort=9 velocity=5 -> lower=-2.79 upper=2.79 effort=20 velocity=5
- joint J2_JOINT: limit lower=-3.14 upper=0 effort=9 velocity=20 -> lower=-3.14 upper=0 effort=20 velocity=5
- joint J3_JOINT: limit lower=0 upper=3.14 effort=9 velocity=20 -> lower=0 upper=3.14 effort=20 velocity=5
- joint J4_JOINT: limit lower=-1.74 upper=1.74 effort=3 velocity=5 -> lower=-1.74 upper=1.74 effort=10 velocity=20
- joint J5_JOINT: limit lower=-1.74 upper=1.74 effort=3 velocity=5 -> lower=-1.74 upper=1.74 effort=10 velocity=20
- joint J6_JOINT: limit lower=-2.61 upper=2.61 effort=3 velocity=5 -> lower=-2.61 upper=2.61 effort=10 velocity=20
