Commit message: fix urdf for ik

File: src/imeta_y1_controller/urdf/y10804.urdf (robot description, URDF)
Before this commit: robot y1, 8 links, 7 joints
Joints:
- joint JOINT1: limit lower=-2.79 upper=2.79 effort=20 velocity=5 -> lower=-3.0 upper=3.0 effort=30 velocity=5
- joint JOINT2: limit lower=-3.14 upper=0 effort=50 velocity=5 -> lower=-3.5 upper=0.2 effort=100 velocity=5
- joint JOINT3: limit lower=0 upper=3.14 effort=20 velocity=5 -> lower=-0.2 upper=4.1 effort=30 velocity=5
- joint JOINT4: limit lower=-1.74 upper=1.74 effort=10 velocity=20 -> lower=-2.5 upper=1.7 effort=10 velocity=20
- joint JOINT5: limit lower=-1.74 upper=1.74 effort=10 velocity=20 -> lower=-2.0 upper=2.0 effort=10 velocity=20
- joint JOINT6: limit lower=-2.61 upper=2.61 effort=10 velocity=20 -> lower=-3.0 upper=3.0 effort=10 velocity=20

Commit message: fix Link4 mass

File: src/imeta_y1_controller/urdf/y10804.urdf (robot description, URDF)
Before this commit: robot y1, 8 links, 7 joints
Links:
- link Link3: mass 0.779000 -> 0.84000
Joints:
- joint JOINT1: limit lower=-3.0 upper=3.0 effort=30 velocity=5 -> lower=-2.79 upper=2.79 effort=20 velocity=5
- joint JOINT2: limit lower=-3.5 upper=0.2 effort=100 velocity=5 -> lower=-3.14 upper=0 effort=50 velocity=5
- joint JOINT3: limit lower=-0.2 upper=4.1 effort=30 velocity=5 -> lower=0 upper=3.14 effort=20 velocity=5
- joint JOINT4: limit lower=-2.5 upper=1.7 effort=10 velocity=20 -> lower=-1.74 upper=1.74 effort=10 velocity=20
- joint JOINT5: limit lower=-2.0 upper=2.0 effort=10 velocity=20 -> lower=-1.74 upper=1.74 effort=10 velocity=20
- joint JOINT6: limit lower=-3.0 upper=3.0 effort=10 velocity=20 -> lower=-2.61 upper=2.61 effort=10 velocity=20
