Commit message: fix gazebo load robot

File: src/y1_description/urdf/y1.urdf (robot description, URDF)
Before this commit: robot y1, 7 links, 6 joints
Links:
- removed link J6_Link
- added link world
Joints:
- removed joint J6_JOINT
- added joint fixed_base_joint: type fixed, parent world, child base_link

File: src/y1_description/urdf/y1_gazebo.xacro (robot description, xacro)
@@ -6,6 +6,6 @@
   <link name="world"/>
   <joint name="fixed_base_joint" type="fixed">
-      <parent link="world"/>
-      <child link="base_link"/>
+    <parent link="world"/>
+    <child link="base_link"/>
   </joint>
   <!-- y1 -->
@@ -105,5 +105,5 @@
       lower="-2.79"
       upper="2.79"
-      effort="9"
+      effort="100"
       velocity="5" />
   </joint>
@@ -163,6 +163,6 @@
       lower="-3.14"
       upper="0"
-      effort="0"
-      velocity="0" />
+      effort="100"
+      velocity="5" />
   </joint>
   <link
@@ -221,6 +221,6 @@
       lower="0"
       upper="3.14"
-      effort="0"
-      velocity="0" />
+      effort="100"
+      velocity="5" />
   </joint>
   <link
@@ -279,6 +279,6 @@
       lower="-1.74"
       upper="1.74"
-      effort="0"
-      velocity="0" />
+      effort="100"
+      velocity="5" />
   </joint>
   <link
@@ -337,8 +337,8 @@
       lower="-1.74"
       upper="1.74"
-      effort="0"
-      velocity="0" />
-  </joint>
-  <link
+      effort="100"
+      velocity="5" />
+  </joint>
+  <!-- <link
     name="J6_Link">
     <inertial>
@@ -395,7 +395,7 @@
       lower="-2.61"
       upper="2.61"
-      effort="0"
-      velocity="0" />
-  </joint>
+      effort="100"
+      velocity="5" />
+  </joint> -->
   <!-- controller -->
   <xacro:macro name="transmission_block" params="tran_name joint_name motor_name">
@@ -416,5 +416,5 @@
   <xacro:transmission_block tran_name="tran4" joint_name="J4_JOINT" motor_name="motor4"/>
   <xacro:transmission_block tran_name="tran5" joint_name="J5_JOINT" motor_name="motor5"/>
-  <xacro:transmission_block tran_name="tran6" joint_name="J6_JOINT" motor_name="motor6"/>
+  <!-- <xacro:transmission_block tran_name="tran6" joint_name="J6_JOINT" motor_name="motor6"/> -->
   <!-- <xacro:transmission_block tran_name="tran7" joint_name="joint7" motor_name="motor7"/> -->
   <!-- <xacro:transmission_block tran_name="tran8" joint_name="joint8" motor_name="motor8"/> -->
@@ -426,5 +426,5 @@
     </plugin>
   </gazebo>
-  <gazebo reference="J1_JOINT">
+  <!-- <gazebo reference="J1_JOINT">
     <provideFeedback>true</provideFeedback>
   </gazebo>
@@ -475,6 +475,6 @@
       <jointName>J5_JOINT</jointName>
     </plugin>
-  </gazebo>
-  <gazebo reference="J6_JOINT">
+  </gazebo> -->
+  <!-- <gazebo reference="J6_JOINT">
     <provideFeedback>true</provideFeedback>
   </gazebo>
@@ -485,4 +485,4 @@
       <jointName>J6_JOINT</jointName>
     </plugin>
-  </gazebo>
+  </gazebo> -->
 </robot>

Commit message: update 20250616 new urdf

File: src/y1_description/urdf/y1.urdf (robot description, URDF)
Before this commit: robot y1, 7 links, 6 joints
Links:
- added link J6_Link, mass 0.8; collision mesh filename=package://y1_description/meshes/J6_Link.STL; visual mesh filename=package://y1_description/meshes/J6_Link.STL
Joints:
- added joint J6_JOINT: type revolute, parent J5_Link, child J6_Link, origin xyz=0.020033 0 0.033914 rpy=1.5466 1.5708 1.5466, axis 0 0 1, limit lower=-2.61 upper=2.61 effort=3 velocity=5
- joint J2_JOINT: limit lower=-3.14 upper=0 effort=0 velocity=0 -> lower=-3.14 upper=0 effort=9 velocity=20; origin xyz=0 0 0.055 rpy=-1.5707963267949 0 0 -> xyz=0 0 0.055 rpy=-1.5708 0 0
- joint J3_JOINT: limit lower=0 upper=3.14 effort=0 velocity=0 -> lower=0 upper=3.14 effort=9 velocity=20
- joint J4_JOINT: limit lower=-1.74 upper=1.74 effort=0 velocity=0 -> lower=-1.74 upper=1.74 effort=3 velocity=5; origin xyz=-0.2140106932061 -0.05098453876871 0 rpy=0 0 0 -> xyz=-0.21401 -0.050985 0 rpy=0 0 0
- joint J5_JOINT: axis 0 0 -1 -> 0 0 1; limit lower=-1.74 upper=1.74 effort=0 velocity=0 -> lower=-1.74 upper=1.74 effort=3 velocity=5; origin xyz=-0.0722997230374954 -0.0454899000967161 0 rpy=1.5707963267949 0 0.0872664625997022 -> xyz=-0.0723 -0.04549 0 rpy=1.5708 0 -3.0543

File: src/y1_description/urdf/y1_gazebo.xacro (robot description, xacro)
@@ -105,5 +105,5 @@
       lower="-2.79"
       upper="2.79"
-      effort="100"
+      effort="9"
       velocity="5" />
   </joint>
@@ -153,5 +153,5 @@
     <origin
       xyz="0 0 0.055"
-      rpy="-1.5707963267949 0 0" />
+      rpy="-1.5708 0 0" />
     <parent
       link="J1_Link" />
@@ -163,6 +163,6 @@
       lower="-3.14"
       upper="0"
-      effort="100"
-      velocity="5" />
+      effort="9"
+      velocity="20" />
   </joint>
   <link
@@ -221,6 +221,6 @@
       lower="0"
       upper="3.14"
-      effort="100"
-      velocity="5" />
+      effort="9"
+      velocity="20" />
   </joint>
   <link
@@ -268,5 +268,5 @@
     type="revolute">
     <origin
-      xyz="-0.2140106932061 -0.05098453876871 0"
+      xyz="-0.21401 -0.050985 0"
       rpy="0 0 0" />
     <parent
@@ -279,5 +279,5 @@
       lower="-1.74"
       upper="1.74"
-      effort="100"
+      effort="3"
       velocity="5" />
   </joint>
@@ -286,5 +286,5 @@
     <inertial>
       <origin
-        xyz="-0.006836 3.7476E-05 -0.027245"
+        xyz="0.006836 3.7476E-05 0.027245"
         rpy="0 0 0" />
       <mass
@@ -292,8 +292,8 @@
       <inertia
         ixx="8.168E-05"
-        ixy="3.1597E-08"
+        ixy="-3.1597E-08"
         ixz="9.4321E-06"
         iyy="6.5589E-05"
-        iyz="1.5004E-08"
+        iyz="-1.5004E-08"
         izz="5.7856E-05" />
     </inertial>
@@ -326,6 +326,6 @@
     type="revolute">
     <origin
-      xyz="-0.0722997230374954 -0.0454899000967161 0"
-      rpy="1.5707963267949 0 0.0872664625997022" />
+      xyz="-0.0723 -0.04549 0"
+      rpy="1.5708 0 -3.0543" />
     <parent
       link="J4_Link" />
@@ -333,9 +333,9 @@
       link="J5_Link" />
     <axis
-      xyz="0 0 -1" />
+      xyz="0 0 1" />
     <limit
       lower="-1.74"
       upper="1.74"
-      effort="100"
+      effort="3"
       velocity="5" />
   </joint>
@@ -347,5 +347,5 @@
         rpy="0 0 0" />
       <mass
-        value="0.8968" />
+        value="0.8" />
       <inertia
         ixx="0.051146"
@@ -384,6 +384,6 @@
     type="revolute">
     <origin
-      xyz="-0.0200325738541419 0 -0.0339137808775768"
-      rpy="3.14159263868863 -1.5707963267949 0" />
+      xyz="0.020033 0 0.033914"
+      rpy="1.5466 1.5708 1.5466" />
     <parent
       link="J5_Link" />
@@ -391,9 +391,9 @@
       link="J6_Link" />
     <axis
-      xyz="0 0 -1" />
+      xyz="0 0 1" />
     <limit
       lower="-2.61"
       upper="2.61"
-      effort="100"
+      effort="3"
       velocity="5" />
   </joint> -->
@@ -426,5 +426,5 @@
     </plugin>
   </gazebo>
-  <!-- <gazebo reference="J1_JOINT">
+  <gazebo reference="J1_JOINT">
     <provideFeedback>true</provideFeedback>
   </gazebo>
@@ -475,5 +475,5 @@
       <jointName>J5_JOINT</jointName>
     </plugin>
-  </gazebo> -->
+  </gazebo>
   <!-- <gazebo reference="J6_JOINT">
     <provideFeedback>true</provideFeedback>

Commit message: fix urdf with ee

File: src/y1_description/urdf/y1.urdf (robot description, URDF)
Before this commit: robot y1, 8 links, 7 joints
Links:
- removed link J1_Link
- removed link J2_Link
- removed link J3_Link
- removed link J4_Link
- removed link J5_Link
- removed link J6_Link
- added link Claw_Link_L, mass 0.086; collision mesh filename=package://y1_description/meshes/Claw_Link_L.STL; visual mesh filename=package://y1_description/meshes/Claw_Link_L.STL
- added link Claw_Link_R, mass 0.086; collision mesh filename=package://y1_description/meshes/Claw_Link_R.STL; visual mesh filename=package://y1_description/meshes/Claw_Link_R.STL
- added link Link1, mass 0.893000; collision mesh filename=package://y1_description/meshes/Link1.STL; visual mesh filename=package://y1_description/meshes/Link1.STL
- added link Link2, mass 1.028000; collision mesh filename=package://y1_description/meshes/Link2.STL; visual mesh filename=package://y1_description/meshes/Link2.STL
- added link Link3, mass 0.838; collision mesh filename=package://y1_description/meshes/Link3.STL; visual mesh filename=package://y1_description/meshes/Link3.STL
- added link Link4, mass 0.444000; collision mesh filename=package://y1_description/meshes/Link4.STL; visual mesh filename=package://y1_description/meshes/Link4.STL
- added link Link5, mass 0.363000; collision mesh filename=package://y1_description/meshes/Link5.STL; visual mesh filename=package://y1_description/meshes/Link5.STL
- added link Link6, mass  0.479; collision mesh filename=package://y1_description/meshes/Link6.STL; visual mesh filename=package://y1_description/meshes/Link6.STL
- link base_link: mass 1.55068784468738 -> 0.632
Joints:
- removed joint J1_JOINT
- removed joint J2_JOINT
- removed joint J3_JOINT
- removed joint J4_JOINT
- removed joint J5_JOINT
- removed joint J6_JOINT
- added joint Claw_Link_L: type prismatic, parent Link6, child Claw_Link_L, origin xyz=-0.0012063 -0.077001 0.07579 rpy=0 -1.5708 -1.5708, axis 0 0 -1, limit lower=0 upper=0.045 effort=10 velocity=20
- added joint Claw_Link_R: type prismatic, parent Link6, child Claw_Link_R, origin xyz=-0.0012063 0.076999 0.075791 rpy=0 -1.5708 -1.5708, axis 0 0 -1, limit lower=0 upper=0.045 effort=10 velocity=20
- added joint JOINT1: type revolute, parent base_link, child Link1, origin xyz=0 0 0 rpy=0 0 0, axis 0 0 -1, limit lower=-3.0 upper=3.0 effort=30 velocity=5
- added joint JOINT2: type revolute, parent Link1, child Link2, origin xyz=0.00075 0 0.055 rpy=1.5708 0 0, axis 0 0 1, limit lower=-3.5 upper=0.2 effort=100 velocity=5
- added joint JOINT3: type revolute, parent Link2, child Link3, origin xyz=-0.28 0 0 rpy=0 0 0, axis 0 0 1, limit lower=-0.2 upper=4.1 effort=30 velocity=5
- added joint JOINT4: type revolute, parent Link3, child Link4, origin xyz=0.215 0.063 0 rpy=0 0 0, axis 0 0 1, limit lower=-2.5 upper=1.7 effort=10 velocity=20
- added joint JOINT5: type revolute, parent Link4, child Link5, origin xyz=0.080817 0.05072 0.00025 rpy=1.5708 0 -0.015918, axis 0 0 1, limit lower=-2.0 upper=2.0 effort=10 velocity=20
- added joint JOINT6: type revolute, parent Link5, child Link6, origin xyz=0.0235 0 0.044 rpy=3.1416 1.5708 3.1416, axis 0 0 1, limit lower=-3.0 upper=3.0 effort=10 velocity=20
- joint fixed_base_joint: axis (none) -> 0 0 1; origin (none) -> xyz=0 0 0.06675 rpy=0 0 0

File: src/y1_description/urdf/y1_gazebo.xacro (robot description, xacro)
@@ -6,6 +6,11 @@
   <link name="world"/>
   <joint name="fixed_base_joint" type="fixed">
+    <origin
+      xyz="0 0 0.08475"
+      rpy="0 0 0" />
     <parent link="world"/>
     <child link="base_link"/>
+    <axis
+      xyz="0 0 1" />
   </joint>
   <!-- y1 -->

Commit message: add y1_sim.

File: src/y1_description/urdf/y1.urdf (robot description, URDF)
Before this commit: robot y1, 10 links, 9 joints
Links:
- removed link Claw_Link_L
- removed link Claw_Link_R
- removed link Link1
- removed link Link2
- removed link Link3
- removed link Link4
- removed link Link5
- removed link Link6
- added link link1, mass 0.893000; collision mesh filename=package://y1_description/meshes1/link1.STL; visual mesh filename=package://y1_description/meshes1/link1.STL
- added link link2, mass 1.028000; collision mesh filename=package://y1_description/meshes1/link2.STL; visual mesh filename=package://y1_description/meshes1/link2.STL
- added link link3, mass 0.84000; collision mesh filename=package://y1_description/meshes1/link3.STL; visual mesh filename=package://y1_description/meshes1/link3.STL
- added link link4, mass 0.444000; collision mesh filename=package://y1_description/meshes1/link4.STL; visual mesh filename=package://y1_description/meshes1/link4.STL
- added link link5, mass 0.363000; collision mesh filename=package://y1_description/meshes1/link5.STL; visual mesh filename=package://y1_description/meshes1/link5.STL
- added link link6, mass 0.016469; collision mesh filename=package://y1_description/meshes1/link6.STL; visual mesh filename=package://y1_description/meshes1/link6.STL
- link base_link: geometry collision mesh filename=package://y1_description/meshes1/base_link.STL; visual mesh filename=package://y1_description/meshes1/base_link.STL
Joints:
- removed joint Claw_Link_L
- removed joint Claw_Link_R
- removed joint JOINT1
- removed joint JOINT2
- removed joint JOINT3
- removed joint JOINT4
- removed joint JOINT5
- removed joint JOINT6
- added joint joint1: type revolute, parent base_link, child link1, origin xyz=0 0 0.06675 rpy=0 0 0, axis 0 0 -1, limit lower=-2.8 upper=2.8 effort=30 velocity=5
- added joint joint2: type revolute, parent link1, child link2, origin xyz=0.00075 0 0.055 rpy=1.5708 0 0, axis 0 0 1, limit lower=-3.23 upper=0.0 effort=100 velocity=5
- added joint joint3: type revolute, parent link2, child link3, origin xyz=-0.28 0 0 rpy=0 0 0, axis 0 0 1, limit lower=0.0 upper=3.05 effort=30 velocity=5
- added joint joint4: type revolute, parent link3, child link4, origin xyz=0.215 0.063 0 rpy=0 0 0, axis 0 0 1, limit lower=-2.1 upper=1.4 effort=30 velocity=5
- added joint joint5: type revolute, parent link4, child link5, origin xyz=0.080817 0.05072 0.00025 rpy=1.5708 0 -0.015918, axis 0 0 1, limit lower=-1.4 upper=1.4 effort=10 velocity=20
- added joint joint6: type revolute, parent link5, child link6, origin xyz=0.0235 0 0.044 rpy=3.1416 1.5708 3.1416, axis 0 0 1, limit lower=-2.5 upper=2.5 effort=10 velocity=20
- joint fixed_base_joint: axis 0 0 1 -> (none); origin xyz=0 0 0.06675 rpy=0 0 0 -> (none)
