Commit message: fix moveit&rviz&gzebo.

File: src/y1_description/urdf/y1_no_gripper.urdf (robot description, URDF)
Before this commit: robot y1, 8 links, 7 joints
Links:
- removed link Link1
- removed link Link2
- removed link Link3
- removed link Link4
- removed link Link5
- removed link Link6
- added link link1, mass 0.465086237348566; collision mesh filename=package://y1_description/meshes/link1.STL; visual mesh filename=package://y1_description/meshes/link1.STL
- added link link2, mass 1.00848298846255; collision mesh filename=package://y1_description/meshes/link2.STL; visual mesh filename=package://y1_description/meshes/link2.STL
- added link link3, mass 0.839664047451371; collision mesh filename=package://y1_description/meshes/link3.STL; visual mesh filename=package://y1_description/meshes/link3.STL
- added link link4, mass 0.455192806560725; collision mesh filename=package://y1_description/meshes/link4.STL; visual mesh filename=package://y1_description/meshes/link4.STL
- added link link5, mass 0.373508569742983; collision mesh filename=package://y1_description/meshes/link5.STL; visual mesh filename=package://y1_description/meshes/link5.STL
- added link link6, mass 0.0724468602058996; collision mesh filename=package://y1_description/meshes/link6.STL; visual mesh filename=package://y1_description/meshes/link6.STL
Joints:
- removed joint Joint1
- removed joint Joint2
- removed joint Joint3
- removed joint Joint4
- removed joint Joint5
- removed joint Joint6
- added joint joint1: type revolute, parent base_link, child link1, origin xyz=0 0 0.06675 rpy=0 0 0, axis 0 0 1, limit lower=-2.79 upper=2.79 effort=30 velocity=5
- added joint joint2: type revolute, parent link1, child link2, origin xyz=0.00075 0 0.055 rpy=1.5707963267949 0 0, axis 0 0 1, limit lower=-3.14 upper=0 effort=100 velocity=5
- added joint joint3: type revolute, parent link2, child link3, origin xyz=-0.28 0 0 rpy=0 0 0, axis 0 0 1, limit lower=0 upper=3.14 effort=30 velocity=5
- added joint joint4: type revolute, parent link3, child link4, origin xyz=0.215000000000004 0.0630000000000073 0 rpy=0 0 0, axis 0 0 1, limit lower=-2.145 upper=1.413 effort=10 velocity=20
- added joint joint5: type revolute, parent link4, child link5, origin xyz=0.0799999999999998 0.0519999999999981 0.000249997832942123 rpy=1.5707963267949 0 0, axis 0 0 1, limit lower=-1.482 upper=1.482 effort=10 velocity=20
- added joint joint6: type revolute, parent link5, child link6, origin xyz=0.0235 0 0.0440000000000001 rpy=-3.14159265330655 0 0, axis 1 0 0, limit lower=-2.529 upper=2.529 effort=10 velocity=20

File: src/y1_description/urdf/y1_no_gripper.xacro (robot description, xacro)
@@ -4,5 +4,6 @@
      For more information, please see http://wiki.ros.org/sw_urdf_exporter -->
 <robot
-  name="y1">
+  name="y1"
+  xmlns:xacro="http://ros.org/wiki/xacro">
   <link name="world"/>
   <joint name="fixed_base_joint" type="fixed">
@@ -56,5 +57,5 @@
   </link>
   <link
-    name="Link1">
+    name="link1">
     <inertial>
       <origin
@@ -77,24 +78,24 @@
       <geometry>
         <mesh
-          filename="package://y1_description/meshes/Link1.STL" />
-      </geometry>
-      <material
-        name="">
-        <color
-          rgba="0.898039215686275 0.917647058823529 0.929411764705882 1" />
-      </material>
-    </visual>
-    <collision>
-      <origin
-        xyz="0 0 0"
-        rpy="0 0 0" />
-      <geometry>
-        <mesh
-          filename="package://y1_description/meshes/Link1.STL" />
-      </geometry>
-    </collision>
-  </link>
-  <joint
-    name="Joint1"
+          filename="package://y1_description/meshes/link1.STL" />
+      </geometry>
+      <material
+        name="">
+        <color
+          rgba="0.898039215686275 0.917647058823529 0.929411764705882 1" />
+      </material>
+    </visual>
+    <collision>
+      <origin
+        xyz="0 0 0"
+        rpy="0 0 0" />
+      <geometry>
+        <mesh
+          filename="package://y1_description/meshes/link1.STL" />
+      </geometry>
+    </collision>
+  </link>
+  <joint
+    name="joint1"
     type="revolute">
     <origin
@@ -104,5 +105,5 @@
       link="base_link" />
     <child
-      link="Link1" />
+      link="link1" />
     <axis
       xyz="0 0 1" />
@@ -114,5 +115,5 @@
   </joint>
   <link
-    name="Link2">
+    name="link2">
     <inertial>
       <origin
@@ -135,24 +136,24 @@
       <geometry>
         <mesh
-          filename="package://y1_description/meshes/Link2.STL" />
-      </geometry>
-      <material
-        name="">
-        <color
-          rgba="0.898039215686275 0.917647058823529 0.929411764705882 1" />
-      </material>
-    </visual>
-    <collision>
-      <origin
-        xyz="0 0 0"
-        rpy="0 0 0" />
-      <geometry>
-        <mesh
-          filename="package://y1_description/meshes/Link2.STL" />
-      </geometry>
-    </collision>
-  </link>
-  <joint
-    name="Joint2"
+          filename="package://y1_description/meshes/link2.STL" />
+      </geometry>
+      <material
+        name="">
+        <color
+          rgba="0.898039215686275 0.917647058823529 0.929411764705882 1" />
+      </material>
+    </visual>
+    <collision>
+      <origin
+        xyz="0 0 0"
+        rpy="0 0 0" />
+      <geometry>
+        <mesh
+          filename="package://y1_description/meshes/link2.STL" />
+      </geometry>
+    </collision>
+  </link>
+  <joint
+    name="joint2"
     type="revolute">
     <origin
@@ -160,7 +161,7 @@
       rpy="1.5707963267949 0 0" />
     <parent
-      link="Link1" />
-    <child
-      link="Link2" />
+      link="link1" />
+    <child
+      link="link2" />
     <axis
       xyz="0 0 1" />
@@ -172,5 +173,5 @@
   </joint>
   <link
-    name="Link3">
+    name="link3">
     <inertial>
       <origin
@@ -193,24 +194,24 @@
       <geometry>
         <mesh
-          filename="package://y1_description/meshes/Link3.STL" />
-      </geometry>
-      <material
-        name="">
-        <color
-          rgba="0.898039215686275 0.917647058823529 0.929411764705882 1" />
-      </material>
-    </visual>
-    <collision>
-      <origin
-        xyz="0 0 0"
-        rpy="0 0 0" />
-      <geometry>
-        <mesh
-          filename="package://y1_description/meshes/Link3.STL" />
-      </geometry>
-    </collision>
-  </link>
-  <joint
-    name="Joint3"
+          filename="package://y1_description/meshes/link3.STL" />
+      </geometry>
+      <material
+        name="">
+        <color
+          rgba="0.898039215686275 0.917647058823529 0.929411764705882 1" />
+      </material>
+    </visual>
+    <collision>
+      <origin
+        xyz="0 0 0"
+        rpy="0 0 0" />
+      <geometry>
+        <mesh
+          filename="package://y1_description/meshes/link3.STL" />
+      </geometry>
+    </collision>
+  </link>
+  <joint
+    name="joint3"
     type="revolute">
     <origin
@@ -218,7 +219,7 @@
       rpy="0 0 0" />
     <parent
-      link="Link2" />
-    <child
-      link="Link3" />
+      link="link2" />
+    <child
+      link="link3" />
     <axis
       xyz="0 0 1" />
@@ -230,5 +231,5 @@
   </joint>
   <link
-    name="Link4">
+    name="link4">
     <inertial>
       <origin
@@ -251,24 +252,24 @@
       <geometry>
         <mesh
-          filename="package://y1_description/meshes/Link4.STL" />
-      </geometry>
-      <material
-        name="">
-        <color
-          rgba="0.898039215686275 0.917647058823529 0.929411764705882 1" />
-      </material>
-    </visual>
-    <collision>
-      <origin
-        xyz="0 0 0"
-        rpy="0 0 0" />
-      <geometry>
-        <mesh
-          filename="package://y1_description/meshes/Link4.STL" />
-      </geometry>
-    </collision>
-  </link>
-  <joint
-    name="Joint4"
+          filename="package://y1_description/meshes/link4.STL" />
+      </geometry>
+      <material
+        name="">
+        <color
+          rgba="0.898039215686275 0.917647058823529 0.929411764705882 1" />
+      </material>
+    </visual>
+    <collision>
+      <origin
+        xyz="0 0 0"
+        rpy="0 0 0" />
+      <geometry>
+        <mesh
+          filename="package://y1_description/meshes/link4.STL" />
+      </geometry>
+    </collision>
+  </link>
+  <joint
+    name="joint4"
     type="revolute">
     <origin
@@ -276,7 +277,7 @@
       rpy="0 0 0" />
     <parent
-      link="Link3" />
-    <child
-      link="Link4" />
+      link="link3" />
+    <child
+      link="link4" />
     <axis
       xyz="0 0 1" />
@@ -288,5 +289,5 @@
   </joint>
   <link
-    name="Link5">
+    name="link5">
     <inertial>
       <origin
@@ -309,24 +310,24 @@
       <geometry>
         <mesh
-          filename="package://y1_description/meshes/Link5.STL" />
-      </geometry>
-      <material
-        name="">
-        <color
-          rgba="0.898039215686275 0.917647058823529 0.929411764705882 1" />
-      </material>
-    </visual>
-    <collision>
-      <origin
-        xyz="0 0 0"
-        rpy="0 0 0" />
-      <geometry>
-        <mesh
-          filename="package://y1_description/meshes/Link5.STL" />
-      </geometry>
-    </collision>
-  </link>
-  <joint
-    name="Joint5"
+          filename="package://y1_description/meshes/link5.STL" />
+      </geometry>
+      <material
+        name="">
+        <color
+          rgba="0.898039215686275 0.917647058823529 0.929411764705882 1" />
+      </material>
+    </visual>
+    <collision>
+      <origin
+        xyz="0 0 0"
+        rpy="0 0 0" />
+      <geometry>
+        <mesh
+          filename="package://y1_description/meshes/link5.STL" />
+      </geometry>
+    </collision>
+  </link>
+  <joint
+    name="joint5"
     type="revolute">
     <origin
@@ -334,7 +335,7 @@
       rpy="1.5707963267949 0 0" />
     <parent
-      link="Link4" />
-    <child
-      link="Link5" />
+      link="link4" />
+    <child
+      link="link5" />
     <axis
       xyz="0 0 1" />
@@ -346,5 +347,5 @@
   </joint>
   <link
-    name="Link6">
+    name="link6">
     <inertial>
       <origin
@@ -367,24 +368,24 @@
       <geometry>
         <mesh
-          filename="package://y1_description/meshes/Link6.STL" />
-      </geometry>
-      <material
-        name="">
-        <color
-          rgba="0.898039215686275 0.917647058823529 0.929411764705882 1" />
-      </material>
-    </visual>
-    <collision>
-      <origin
-        xyz="0 0 0"
-        rpy="0 0 0" />
-      <geometry>
-        <mesh
-          filename="package://y1_description/meshes/Link6.STL" />
-      </geometry>
-    </collision>
-  </link>
-  <joint
-    name="Joint6"
+          filename="package://y1_description/meshes/link6.STL" />
+      </geometry>
+      <material
+        name="">
+        <color
+          rgba="0.898039215686275 0.917647058823529 0.929411764705882 1" />
+      </material>
+    </visual>
+    <collision>
+      <origin
+        xyz="0 0 0"
+        rpy="0 0 0" />
+      <geometry>
+        <mesh
+          filename="package://y1_description/meshes/link6.STL" />
+      </geometry>
+    </collision>
+  </link>
+  <joint
+    name="joint6"
     type="revolute">
     <origin
@@ -392,7 +393,7 @@
       rpy="-3.14159265330655 0 0" />
     <parent
-      link="Link5" />
-    <child
-      link="Link6" />
+      link="link5" />
+    <child
+      link="link6" />
     <axis
       xyz="1 0 0" />

File: src/y1_description/urdf/y1_with_gripper.urdf (robot description, URDF)
Before this commit: robot y1, 11 links, 10 joints
Links:
- removed link Claw_Link_L
- removed link Claw_Link_R
- removed link Link1
- removed link Link2
- removed link Link3
- removed link Link4
- removed link Link5
- removed link Link6
- added link link1, mass 0.465086237348566; collision mesh filename=package://y1_description/meshes/link1.STL; visual mesh filename=package://y1_description/meshes/link1.STL
- added link link2, mass 1.00848298846255; collision mesh filename=package://y1_description/meshes/link2.STL; visual mesh filename=package://y1_description/meshes/link2.STL
- added link link3, mass 0.839664047451371; collision mesh filename=package://y1_description/meshes/link3.STL; visual mesh filename=package://y1_description/meshes/link3.STL
- added link link4, mass 0.455192806560725; collision mesh filename=package://y1_description/meshes/link4.STL; visual mesh filename=package://y1_description/meshes/link4.STL
- added link link5, mass 0.373508569742983; collision mesh filename=package://y1_description/meshes/link5.STL; visual mesh filename=package://y1_description/meshes/link5.STL
- added link link6, mass 0.0724468602058996; collision mesh filename=package://y1_description/meshes/link6.STL; visual mesh filename=package://y1_description/meshes/link6.STL
- added link link7, mass 0.0661690926183051; collision mesh filename=package://y1_description/meshes/link7.STL; visual mesh filename=package://y1_description/meshes/link7.STL
- added link link8, mass 0.0661690929217921; collision mesh filename=package://y1_description/meshes/link8.STL; visual mesh filename=package://y1_description/meshes/link8.STL
Joints:
- removed joint Claw_Link_L
- removed joint Claw_Link_R
- removed joint Joint1
- removed joint Joint2
- removed joint Joint3
- removed joint Joint4
- removed joint Joint5
- removed joint Joint6
- added joint joint1: type revolute, parent base_link, child link1, origin xyz=0 0 0.06675 rpy=0 0 0, axis 0 0 1, limit lower=-2.79 upper=2.79 effort=30 velocity=5
- added joint joint2: type revolute, parent link1, child link2, origin xyz=0.00075 0 0.055 rpy=1.5707963267949 0 0, axis 0 0 1, limit lower=-3.14 upper=0 effort=100 velocity=5
- added joint joint3: type revolute, parent link2, child link3, origin xyz=-0.28 0 0 rpy=0 0 0, axis 0 0 1, limit lower=0 upper=3.14 effort=30 velocity=5
- added joint joint4: type revolute, parent link3, child link4, origin xyz=0.215000000000004 0.0630000000000073 0 rpy=0 0 0, axis 0 0 1, limit lower=-2.145 upper=1.413 effort=10 velocity=20
- added joint joint5: type revolute, parent link4, child link5, origin xyz=0.0799999999999998 0.0519999999999981 0.000249997832942123 rpy=1.5707963267949 0 0, axis 0 0 1, limit lower=-1.482 upper=1.482 effort=10 velocity=20
- added joint joint6: type revolute, parent link5, child link6, origin xyz=0.0235 0 0.0440000000000001 rpy=-3.14159265330655 0 0, axis 1 0 0, limit lower=-2.529 upper=2.529 effort=10 velocity=20
- added joint joint7: type prismatic, parent gripper_base, child link7, origin xyz=0 -0.00275000000000102 0 rpy=0 0 -1.5707963267949, axis 1 0 0, limit lower=-0.05 upper=0 effort=3 velocity=0
- added joint joint8: type prismatic, parent gripper_base, child link8, origin xyz=0 0.00274999999999902 0 rpy=0 0 -1.5707963267949, axis 1 0 0, limit lower=0 upper=0.05 effort=3 velocity=0, mimic joint=joint7 multiplier=-1.0 offset=0.0
- joint gripper_base: parent Link6 -> link6

File: src/y1_description/urdf/y1_with_gripper.xacro (robot description, xacro)
@@ -4,5 +4,6 @@
      For more information, please see http://wiki.ros.org/sw_urdf_exporter -->
 <robot
-  name="y1">
+  name="y1"
+  xmlns:xacro="http://ros.org/wiki/xacro">
   <link name="world"/>
   <joint name="fixed_base_joint" type="fixed">
@@ -56,5 +57,5 @@
   </link>
   <link
-    name="Link1">
+    name="link1">
     <inertial>
       <origin
@@ -77,5 +78,5 @@
       <geometry>
         <mesh
-          filename="package://y1_description/meshes/Link1.STL" />
+          filename="package://y1_description/meshes/link1.STL" />
       </geometry>
       <material
@@ -91,10 +92,10 @@
       <geometry>
         <mesh
-          filename="package://y1_description/meshes/Link1.STL" />
-      </geometry>
-    </collision>
-  </link>
-  <joint
-    name="Joint1"
+          filename="package://y1_description/meshes/link1.STL" />
+      </geometry>
+    </collision>
+  </link>
+  <joint
+    name="joint1"
     type="revolute">
     <origin
@@ -104,5 +105,5 @@
       link="base_link" />
     <child
-      link="Link1" />
+      link="link1" />
     <axis
       xyz="0 0 1" />
@@ -114,5 +115,5 @@
   </joint>
   <link
-    name="Link2">
+    name="link2">
     <inertial>
       <origin
@@ -135,5 +136,5 @@
       <geometry>
         <mesh
-          filename="package://y1_description/meshes/Link2.STL" />
+          filename="package://y1_description/meshes/link2.STL" />
       </geometry>
       <material
@@ -149,10 +150,10 @@
       <geometry>
         <mesh
-          filename="package://y1_description/meshes/Link2.STL" />
-      </geometry>
-    </collision>
-  </link>
-  <joint
-    name="Joint2"
+          filename="package://y1_description/meshes/link2.STL" />
+      </geometry>
+    </collision>
+  </link>
+  <joint
+    name="joint2"
     type="revolute">
     <origin
@@ -160,7 +161,7 @@
       rpy="1.5707963267949 0 0" />
     <parent
-      link="Link1" />
-    <child
-      link="Link2" />
+      link="link1" />
+    <child
+      link="link2" />
     <axis
       xyz="0 0 1" />
@@ -172,5 +173,5 @@
   </joint>
   <link
-    name="Link3">
+    name="link3">
     <inertial>
       <origin
@@ -193,5 +194,5 @@
       <geometry>
         <mesh
-          filename="package://y1_description/meshes/Link3.STL" />
+          filename="package://y1_description/meshes/link3.STL" />
       </geometry>
       <material
@@ -207,10 +208,10 @@
       <geometry>
         <mesh
-          filename="package://y1_description/meshes/Link3.STL" />
-      </geometry>
-    </collision>
-  </link>
-  <joint
-    name="Joint3"
+          filename="package://y1_description/meshes/link3.STL" />
+      </geometry>
+    </collision>
+  </link>
+  <joint
+    name="joint3"
     type="revolute">
     <origin
@@ -218,7 +219,7 @@
       rpy="0 0 0" />
     <parent
-      link="Link2" />
-    <child
-      link="Link3" />
+      link="link2" />
+    <child
+      link="link3" />
     <axis
       xyz="0 0 1" />
@@ -230,5 +231,5 @@
   </joint>
   <link
-    name="Link4">
+    name="link4">
     <inertial>
       <origin
@@ -251,5 +252,5 @@
       <geometry>
         <mesh
-          filename="package://y1_description/meshes/Link4.STL" />
+          filename="package://y1_description/meshes/link4.STL" />
       </geometry>
       <material
@@ -265,10 +266,10 @@
       <geometry>
         <mesh
-          filename="package://y1_description/meshes/Link4.STL" />
-      </geometry>
-    </collision>
-  </link>
-  <joint
-    name="Joint4"
+          filename="package://y1_description/meshes/link4.STL" />
+      </geometry>
+    </collision>
+  </link>
+  <joint
+    name="joint4"
     type="revolute">
     <origin
@@ -276,7 +277,7 @@
       rpy="0 0 0" />
     <parent
-      link="Link3" />
-    <child
-      link="Link4" />
+      link="link3" />
+    <child
+      link="link4" />
     <axis
       xyz="0 0 1" />
@@ -288,5 +289,5 @@
   </joint>
   <link
-    name="Link5">
+    name="link5">
     <inertial>
       <origin
@@ -309,5 +310,5 @@
       <geometry>
         <mesh
-          filename="package://y1_description/meshes/Link5.STL" />
+          filename="package://y1_description/meshes/link5.STL" />
       </geometry>
       <material
@@ -323,10 +324,10 @@
       <geometry>
         <mesh
-          filename="package://y1_description/meshes/Link5.STL" />
-      </geometry>
-    </collision>
-  </link>
-  <joint
-    name="Joint5"
+          filename="package://y1_description/meshes/link5.STL" />
+      </geometry>
+    </collision>
+  </link>
+  <joint
+    name="joint5"
     type="revolute">
     <origin
@@ -334,7 +335,7 @@
       rpy="1.5707963267949 0 0" />
     <parent
-      link="Link4" />
-    <child
-      link="Link5" />
+      link="link4" />
+    <child
+      link="link5" />
     <axis
       xyz="0 0 1" />
@@ -346,5 +347,5 @@
   </joint>
   <link
-    name="Link6">
+    name="link6">
     <inertial>
       <origin
@@ -367,5 +368,5 @@
       <geometry>
         <mesh
-          filename="package://y1_description/meshes/Link6.STL" />
+          filename="package://y1_description/meshes/link6.STL" />
       </geometry>
       <material
@@ -381,10 +382,10 @@
       <geometry>
         <mesh
-          filename="package://y1_description/meshes/Link6.STL" />
-      </geometry>
-    </collision>
-  </link>
-  <joint
-    name="Joint6"
+          filename="package://y1_description/meshes/link6.STL" />
+      </geometry>
+    </collision>
+  </link>
+  <joint
+    name="joint6"
     type="revolute">
     <origin
@@ -392,7 +393,7 @@
       rpy="-3.14159265330655 0 0" />
     <parent
-      link="Link5" />
-    <child
-      link="Link6" />
+      link="link5" />
+    <child
+      link="link6" />
     <axis
       xyz="1 0 0" />
@@ -450,5 +451,5 @@
       rpy="1.57079745225378 -1.57079631189374 1.57079520133601" />
     <parent
-      link="Link6" />
+      link="link6" />
     <child
       link="gripper_base" />
@@ -457,5 +458,5 @@
   </joint>
   <link
-    name="Claw_Link_L">
+    name="link7">
     <inertial>
       <origin
@@ -478,5 +479,5 @@
       <geometry>
         <mesh
-          filename="package://y1_description/meshes/Claw_Link_L.STL" />
+          filename="package://y1_description/meshes/link7.STL" />
       </geometry>
       <material
@@ -492,10 +493,10 @@
       <geometry>
         <mesh
-          filename="package://y1_description/meshes/Claw_Link_L.STL" />
-      </geometry>
-    </collision>
-  </link>
-  <joint
-    name="Claw_Link_L"
+          filename="package://y1_description/meshes/link7.STL" />
+      </geometry>
+    </collision>
+  </link>
+  <joint
+    name="joint7"
     type="prismatic">
     <origin
@@ -505,15 +506,15 @@
       link="gripper_base" />
     <child
-      link="Claw_Link_L" />
+      link="link7" />
     <axis
       xyz="1 0 0" />
     <limit
-      lower="-0.047"
+      lower="-0.05"
       upper="0"
       effort="3"
-      velocity="0" />
-  </joint>
-  <link
-    name="Claw_Link_R">
+      velocity="5" />
+  </joint>
+  <link
+    name="link8">
     <inertial>
       <origin
@@ -536,5 +537,5 @@
       <geometry>
         <mesh
-          filename="package://y1_description/meshes/Claw_Link_R.STL" />
+          filename="package://y1_description/meshes/link8.STL" />
       </geometry>
       <material
@@ -550,10 +551,10 @@
       <geometry>
         <mesh
-          filename="package://y1_description/meshes/Claw_Link_R.STL" />
-      </geometry>
-    </collision>
-  </link>
-  <joint
-    name="Claw_Link_R"
+          filename="package://y1_description/meshes/link8.STL" />
+      </geometry>
+    </collision>
+  </link>
+  <joint
+    name="joint8"
     type="prismatic">
     <origin
@@ -563,14 +564,15 @@
       link="gripper_base" />
     <child
-      link="Claw_Link_R" />
+      link="link8" />
     <axis
       xyz="1 0 0" />
+    <mimic joint="joint7" multiplier="-1.0" offset="0.0"/>
     <limit
       lower="0"
-      upper="0.047"
+      upper="0.05"
       effort="3"
-      velocity="0" />
-  </joint>
-    <!-- controller -->
+      velocity="5" />
+  </joint>
+  <!-- controller -->
   <xacro:macro name="transmission_block" params="tran_name joint_name motor_name">
     <transmission name="${tran_name}">
