Commit message: fix moveit&rviz&gzebo.

File: src/y1_moveit/y1_with_gripper_moveit/config/gazebo_y1.urdf (robot description, URDF)
Before this commit: robot y1_description, 11 links, 10 joints
Links:
- link base_link: mass 0.710539568297307 -> 0.630484112037129; geometry collision mesh filename=package://y1_description/meshes/base_link.STL; visual mesh filename=package://y1_description/meshes/base_link.STL
- link gripper_base: mass 0.472677133888304 -> 0.436099620967633; geometry collision mesh filename=package://y1_description/meshes/gripper_base.STL; visual mesh filename=package://y1_description/meshes/gripper_base.STL
- link link1: geometry collision mesh filename=package://y1_description/meshes/link1.STL; visual mesh filename=package://y1_description/meshes/link1.STL
- link link2: mass 1.00848298285328 -> 1.00848298846255; geometry collision mesh filename=package://y1_description/meshes/link2.STL; visual mesh filename=package://y1_description/meshes/link2.STL
- link link3: mass 0.839664048562432 -> 0.839664047451371; geometry collision mesh filename=package://y1_description/meshes/link3.STL; visual mesh filename=package://y1_description/meshes/link3.STL
- link link4: mass 0.455192807281481 -> 0.455192806560725; geometry collision mesh filename=package://y1_description/meshes/link4.STL; visual mesh filename=package://y1_description/meshes/link4.STL
- link link5: mass 0.37350857138172 -> 0.373508569742983; geometry collision mesh filename=package://y1_description/meshes/link5.STL; visual mesh filename=package://y1_description/meshes/link5.STL
- link link6: mass 0.0710864913917462 -> 0.0724468602058996; geometry collision mesh filename=package://y1_description/meshes/link6.STL; visual mesh filename=package://y1_description/meshes/link6.STL
- link link7: mass 0.0941874462283945 -> 0.0661690926183051; geometry collision mesh filename=package://y1_description/meshes/link7.STL; visual mesh filename=package://y1_description/meshes/link7.STL
- link link8: mass 0.0941874502574237 -> 0.0661690929217921; geometry collision mesh filename=package://y1_description/meshes/link8.STL; visual mesh filename=package://y1_description/meshes/link8.STL
Joints:
- joint fixed_base_joint: axis (none) -> 0 0 1; origin (none) -> xyz=0 0 0 rpy=0 0 0
- joint gripper_base: origin xyz=-0.00120627967358662 0 0.0757904010332325 rpy=0 -0.015914651654156 0 -> xyz=0.0758 0 0 rpy=1.57079745225378 -1.57079631189374 1.57079520133601
- joint joint1: limit lower=-3.0 upper=3.0 effort=30 velocity=5 -> lower=-2.79 upper=2.79 effort=30 velocity=5
- joint joint2: limit lower=-3.5 upper=0.2 effort=100 velocity=5 -> lower=-3.14 upper=0 effort=100 velocity=5
- joint joint3: limit lower=-0.2 upper=4.1 effort=30 velocity=5 -> lower=0 upper=3.14 effort=30 velocity=5
- joint joint4: limit lower=-2.5 upper=1.7 effort=10 velocity=20 -> lower=-2.145 upper=1.413 effort=10 velocity=20; origin xyz=0.215000000191949 0.062999999344955 0 rpy=0 0 0 -> xyz=0.215000000000004 0.0630000000000073 0 rpy=0 0 0
- joint joint5: limit lower=-2.0 upper=2.0 effort=10 velocity=20 -> lower=-1.482 upper=1.482 effort=10 velocity=20; origin xyz=0.0808173961212753 0.0507202965702747 0.000249997832943334 rpy=1.5707963267949 0 0 -> xyz=0.0799999999999998 0.0519999999999981 0.000249997832942123 rpy=1.5707963267949 0 0
- joint joint6: axis 0 0 1 -> 1 0 0; limit lower=-3.0 upper=3.0 effort=10 velocity=20 -> lower=-2.529 upper=2.529 effort=10 velocity=20; origin xyz=0.0227968089529965 0 0.0443684065693784 rpy=0 1.5707963267949 0 -> xyz=0.0235 0 0.0440000000000001 rpy=-3.14159265330655 0 0
- joint joint7: axis 0 0 -1 -> 1 0 0; limit lower=0 upper=0.04 effort=10 velocity=20 -> lower=-0.05 upper=0 effort=3 velocity=0; origin xyz=0 -0.080000000000001 0 rpy=-1.5707963267949 -1.55488167514075 0 -> xyz=0 -0.00275000000000102 0 rpy=0 0 -1.5707963267949
- joint joint8: axis 0 0 1 -> -1 0 0; limit lower=0 upper=0.04 effort=10 velocity=20 -> lower=0 upper=0.05 effort=3 velocity=0; origin xyz=0 0.08 0 rpy=-1.5708 -1.5549 0 -> xyz=0 0.00274999999999902 0 rpy=0 0 -1.5707963267949
