Commit message: add moveit and gazebo module.

File: src/y1_description/urdf/y1_no_gripper.xacro (robot description, xacro)
@@ -1,6 +1,5 @@
 <?xml version="1.0" encoding="utf-8"?>
-<!-- This URDF was automatically created by SolidWorks to URDF Exporter! Originally created by Stephen Brawner (brawner@gmail.com)
-     Commit Version: 1.6.0-4-g7f85cfe  Build Version: 1.6.7995.38578
-     For more information, please see http://wiki.ros.org/sw_urdf_exporter -->
+<!-- This URDF was automatically created by SolidWorks to URDF Exporter!
+     Modified for ROS 2 (gazebo_ros2_control) -->
 <robot
   name="y1"
@@ -16,6 +15,6 @@
       xyz="0 0 1" />
   </joint>
-  <link
-    name="base_link">
+  <!-- ================= Base Link ================= -->
+  <link name="base_link">
     <inertial>
       <origin
@@ -38,24 +37,24 @@
       <geometry>
         <mesh
-          filename="package://y1_description/meshes/base_link.STL" />
-      </geometry>
-      <material
-        name="">
-        <color
-          rgba="0.898039215686275 0.917647058823529 0.929411764705882 1" />
-      </material>
-    </visual>
-    <collision>
-      <origin
-        xyz="0 0 0"
-        rpy="0 0 0" />
-      <geometry>
-        <mesh
-          filename="package://y1_description/meshes/base_link.STL" />
-      </geometry>
-    </collision>
-  </link>
-  <link
-    name="link1">
+          filename="file://$(find y1_description)/meshes/base_link.STL" />
+      </geometry>
+      <material
+        name="">
+        <color
+          rgba="0.898039215686275 0.917647058823529 0.929411764705882 1" />
+      </material>
+    </visual>
+    <collision>
+      <origin
+        xyz="0 0 0"
+        rpy="0 0 0" />
+      <geometry>
+        <mesh
+          filename="file://$(find y1_description)/meshes/base_link.STL" />
+      </geometry>
+    </collision>
+  </link>
+  <!-- ================= Joint 1 & Link 1 ================= -->
+  <link name="link1">
     <inertial>
       <origin
@@ -78,34 +77,29 @@
       <geometry>
         <mesh
-          filename="package://y1_description/meshes/link1.STL" />
-      </geometry>
-      <material
-        name="">
-        <color
-          rgba="0.898039215686275 0.917647058823529 0.929411764705882 1" />
-      </material>
-    </visual>
-    <collision>
-      <origin
-        xyz="0 0 0"
-        rpy="0 0 0" />
-      <geometry>
-        <mesh
-          filename="package://y1_description/meshes/link1.STL" />
-      </geometry>
-    </collision>
-  </link>
-  <joint
-    name="joint1"
-    type="revolute">
+          filename="file://$(find y1_description)/meshes/link1.STL" />
+      </geometry>
+      <material
+        name="">
+        <color
+          rgba="0.898039215686275 0.917647058823529 0.929411764705882 1" />
+      </material>
+    </visual>
+    <collision>
+      <origin
+        xyz="0 0 0"
+        rpy="0 0 0" />
+      <geometry>
+        <mesh
+          filename="file://$(find y1_description)/meshes/link1.STL" />
+      </geometry>
+    </collision>
+  </link>
+  <joint name="joint1" type="revolute">
     <origin
       xyz="0 0 0.06675"
       rpy="0 0 0" />
-    <parent
-      link="base_link" />
-    <child
-      link="link1" />
-    <axis
-      xyz="0 0 1" />
+    <parent link="base_link" />
+    <child link="link1" />
+    <axis xyz="0 0 1" />
     <limit
       lower="-2.79"
@@ -114,6 +108,6 @@
       velocity="5" />
   </joint>
-  <link
-    name="link2">
+  <!-- ================= Joint 2 & Link 2 ================= -->
+  <link name="link2">
     <inertial>
       <origin
@@ -136,34 +130,29 @@
       <geometry>
         <mesh
-          filename="package://y1_description/meshes/link2.STL" />
-      </geometry>
-      <material
-        name="">
-        <color
-          rgba="0.898039215686275 0.917647058823529 0.929411764705882 1" />
-      </material>
-    </visual>
-    <collision>
-      <origin
-        xyz="0 0 0"
-        rpy="0 0 0" />
-      <geometry>
-        <mesh
-          filename="package://y1_description/meshes/link2.STL" />
-      </geometry>
-    </collision>
-  </link>
-  <joint
-    name="joint2"
-    type="revolute">
+          filename="file://$(find y1_description)/meshes/link2.STL" />
+      </geometry>
+      <material
+        name="">
+        <color
+          rgba="0.898039215686275 0.917647058823529 0.929411764705882 1" />
+      </material>
+    </visual>
+    <collision>
+      <origin
+        xyz="0 0 0"
+        rpy="0 0 0" />
+      <geometry>
+        <mesh
+          filename="file://$(find y1_description)/meshes/link2.STL" />
+      </geometry>
+    </collision>
+  </link>
+  <joint name="joint2" type="revolute">
     <origin
       xyz="0.00075 0 0.055"
       rpy="1.5707963267949 0 0" />
-    <parent
-      link="link1" />
-    <child
-      link="link2" />
-    <axis
-      xyz="0 0 1" />
+    <parent link="link1" />
+    <child link="link2" />
+    <axis xyz="0 0 1" />
     <limit
       lower="-3.14"
@@ -172,6 +161,6 @@
       velocity="5" />
   </joint>
-  <link
-    name="link3">
+  <!-- ================= Joint 3 & Link 3 ================= -->
+  <link name="link3">
     <inertial>
       <origin
@@ -194,34 +183,29 @@
       <geometry>
         <mesh
-          filename="package://y1_description/meshes/link3.STL" />
-      </geometry>
-      <material
-        name="">
-        <color
-          rgba="0.898039215686275 0.917647058823529 0.929411764705882 1" />
-      </material>
-    </visual>
-    <collision>
-      <origin
-        xyz="0 0 0"
-        rpy="0 0 0" />
-      <geometry>
-        <mesh
-          filename="package://y1_description/meshes/link3.STL" />
-      </geometry>
-    </collision>
-  </link>
-  <joint
-    name="joint3"
-    type="revolute">
+          filename="file://$(find y1_description)/meshes/link3.STL" />
+      </geometry>
+      <material
+        name="">
+        <color
+          rgba="0.898039215686275 0.917647058823529 0.929411764705882 1" />
+      </material>
+    </visual>
+    <collision>
+      <origin
+        xyz="0 0 0"
+        rpy="0 0 0" />
+      <geometry>
+        <mesh
+          filename="file://$(find y1_description)/meshes/link3.STL" />
+      </geometry>
+    </collision>
+  </link>
+  <joint name="joint3" type="revolute">
     <origin
       xyz="-0.28 0 0"
       rpy="0 0 0" />
-    <parent
-      link="link2" />
-    <child
-      link="link3" />
-    <axis
-      xyz="0 0 1" />
+    <parent link="link2" />
+    <child link="link3" />
+    <axis xyz="0 0 1" />
     <limit
       lower="0"
@@ -230,6 +214,6 @@
       velocity="5" />
   </joint>
-  <link
-    name="link4">
+  <!-- ================= Joint 4 & Link 4 ================= -->
+  <link name="link4">
     <inertial>
       <origin
@@ -252,34 +236,29 @@
       <geometry>
         <mesh
-          filename="package://y1_description/meshes/link4.STL" />
-      </geometry>
-      <material
-        name="">
-        <color
-          rgba="0.898039215686275 0.917647058823529 0.929411764705882 1" />
-      </material>
-    </visual>
-    <collision>
-      <origin
-        xyz="0 0 0"
-        rpy="0 0 0" />
-      <geometry>
-        <mesh
-          filename="package://y1_description/meshes/link4.STL" />
-      </geometry>
-    </collision>
-  </link>
-  <joint
-    name="joint4"
-    type="revolute">
+          filename="file://$(find y1_description)/meshes/link4.STL" />
+      </geometry>
+      <material
+        name="">
+        <color
+          rgba="0.898039215686275 0.917647058823529 0.929411764705882 1" />
+      </material>
+    </visual>
+    <collision>
+      <origin
+        xyz="0 0 0"
+        rpy="0 0 0" />
+      <geometry>
+        <mesh
+          filename="file://$(find y1_description)/meshes/link4.STL" />
+      </geometry>
+    </collision>
+  </link>
+  <joint name="joint4" type="revolute">
     <origin
       xyz="0.215000000000004 0.0630000000000073 0"
       rpy="0 0 0" />
-    <parent
-      link="link3" />
-    <child
-      link="link4" />
-    <axis
-      xyz="0 0 1" />
+    <parent link="link3" />
+    <child link="link4" />
+    <axis xyz="0 0 1" />
     <limit
       lower="-2.145"
@@ -288,6 +267,6 @@
       velocity="20" />
   </joint>
-  <link
-    name="link5">
+  <!-- ================= Joint 5 & Link 5 ================= -->
+  <link name="link5">
     <inertial>
       <origin
@@ -310,34 +289,29 @@
       <geometry>
         <mesh
-          filename="package://y1_description/meshes/link5.STL" />
-      </geometry>
-      <material
-        name="">
-        <color
-          rgba="0.898039215686275 0.917647058823529 0.929411764705882 1" />
-      </material>
-    </visual>
-    <collision>
-      <origin
-        xyz="0 0 0"
-        rpy="0 0 0" />
-      <geometry>
-        <mesh
-          filename="package://y1_description/meshes/link5.STL" />
-      </geometry>
-    </collision>
-  </link>
-  <joint
-    name="joint5"
-    type="revolute">
+          filename="file://$(find y1_description)/meshes/link5.STL" />
+      </geometry>
+      <material
+        name="">
+        <color
+          rgba="0.898039215686275 0.917647058823529 0.929411764705882 1" />
+      </material>
+    </visual>
+    <collision>
+      <origin
+        xyz="0 0 0"
+        rpy="0 0 0" />
+      <geometry>
+        <mesh
+          filename="file://$(find y1_description)/meshes/link5.STL" />
+      </geometry>
+    </collision>
+  </link>
+  <joint name="joint5" type="revolute">
     <origin
       xyz="0.0799999999999998 0.0519999999999981 0.000249997832942123"
       rpy="1.5707963267949 0 0" />
-    <parent
-      link="link4" />
-    <child
-      link="link5" />
-    <axis
-      xyz="0 0 1" />
+    <parent link="link4" />
+    <child link="link5" />
+    <axis xyz="0 0 1" />
     <limit
       lower="-1.482"
@@ -346,6 +320,6 @@
       velocity="20" />
   </joint>
-  <link
-    name="link6">
+  <!-- ================= Joint 6 & Link 6 ================= -->
+  <link name="link6">
     <inertial>
       <origin
@@ -368,34 +342,29 @@
       <geometry>
         <mesh
-          filename="package://y1_description/meshes/link6.STL" />
-      </geometry>
-      <material
-        name="">
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
File: src/y1_description/urdf/y1_with_gripper.xacro (robot description, xacro)
@@ -4,6 +4,5 @@
      For more information, please see http://wiki.ros.org/sw_urdf_exporter -->
 <robot
-  name="y1"
-  xmlns:xacro="http://ros.org/wiki/xacro">
+  name="y1">
   <link name="world"/>
   <joint name="fixed_base_joint" type="fixed">
@@ -38,5 +37,5 @@
       <geometry>
         <mesh
-          filename="package://y1_description/meshes/base_link.STL" />
+          filename="file://$(find y1_description)/meshes/base_link.STL" />
       </geometry>
       <material
@@ -52,5 +51,5 @@
       <geometry>
         <mesh
-          filename="package://y1_description/meshes/base_link.STL" />
+          filename="file://$(find y1_description)/meshes/base_link.STL" />
       </geometry>
     </collision>
@@ -78,5 +77,5 @@
       <geometry>
         <mesh
-          filename="package://y1_description/meshes/link1.STL" />
+          filename="file://$(find y1_description)/meshes/link1.STL" />
       </geometry>
       <material
@@ -92,5 +91,5 @@
       <geometry>
         <mesh
-          filename="package://y1_description/meshes/link1.STL" />
+          filename="file://$(find y1_description)/meshes/link1.STL" />
       </geometry>
     </collision>
@@ -136,5 +135,5 @@
       <geometry>
         <mesh
-          filename="package://y1_description/meshes/link2.STL" />
+          filename="file://$(find y1_description)/meshes/link2.STL" />
       </geometry>
       <material
@@ -150,5 +149,5 @@
       <geometry>
         <mesh
-          filename="package://y1_description/meshes/link2.STL" />
+          filename="file://$(find y1_description)/meshes/link2.STL" />
       </geometry>
     </collision>
@@ -194,5 +193,5 @@
       <geometry>
         <mesh
-          filename="package://y1_description/meshes/link3.STL" />
+          filename="file://$(find y1_description)/meshes/link3.STL" />
       </geometry>
       <material
@@ -208,5 +207,5 @@
       <geometry>
         <mesh
-          filename="package://y1_description/meshes/link3.STL" />
+          filename="file://$(find y1_description)/meshes/link3.STL" />
       </geometry>
     </collision>
@@ -252,5 +251,5 @@
       <geometry>
         <mesh
-          filename="package://y1_description/meshes/link4.STL" />
+          filename="file://$(find y1_description)/meshes/link4.STL" />
       </geometry>
       <material
@@ -266,5 +265,5 @@
       <geometry>
         <mesh
-          filename="package://y1_description/meshes/link4.STL" />
+          filename="file://$(find y1_description)/meshes/link4.STL" />
       </geometry>
     </collision>
@@ -310,5 +309,5 @@
       <geometry>
         <mesh
-          filename="package://y1_description/meshes/link5.STL" />
+          filename="file://$(find y1_description)/meshes/link5.STL" />
       </geometry>
       <material
@@ -324,5 +323,5 @@
       <geometry>
         <mesh
-          filename="package://y1_description/meshes/link5.STL" />
+          filename="file://$(find y1_description)/meshes/link5.STL" />
       </geometry>
     </collision>
@@ -368,5 +367,5 @@
       <geometry>
         <mesh
-          filename="package://y1_description/meshes/link6.STL" />
+          filename="file://$(find y1_description)/meshes/link6.STL" />
       </geometry>
       <material
@@ -382,5 +381,5 @@
       <geometry>
         <mesh
-          filename="package://y1_description/meshes/link6.STL" />
+          filename="file://$(find y1_description)/meshes/link6.STL" />
       </geometry>
     </collision>
@@ -426,5 +425,5 @@
       <geometry>
         <mesh
-          filename="package://y1_description/meshes/gripper_base.STL" />
+          filename="file://$(find y1_description)/meshes/gripper_base.STL" />
       </geometry>
       <material
@@ -440,5 +439,5 @@
       <geometry>
         <mesh
-          filename="package://y1_description/meshes/gripper_base.STL" />
+          filename="file://$(find y1_description)/meshes/gripper_base.STL" />
       </geometry>
     </collision>
@@ -479,5 +478,5 @@
       <geometry>
         <mesh
-          filename="package://y1_description/meshes/link7.STL" />
+          filename="file://$(find y1_description)/meshes/link7.STL" />
       </geometry>
       <material
@@ -493,5 +492,5 @@
       <geometry>
         <mesh
-          filename="package://y1_description/meshes/link7.STL" />
+          filename="file://$(find y1_description)/meshes/link7.STL" />
       </geometry>
     </collision>
@@ -513,5 +512,5 @@
       upper="0"
       effort="3"
-      velocity="5" />
+      velocity="0" />
   </joint>
   <link
@@ -537,5 +536,5 @@
       <geometry>
         <mesh
-          filename="package://y1_description/meshes/link8.STL" />
+          filename="file://$(find y1_description)/meshes/link8.STL" />
       </geometry>
       <material
@@ -551,5 +550,5 @@
       <geometry>
         <mesh
-          filename="package://y1_description/meshes/link8.STL" />
+          filename="file://$(find y1_description)/meshes/link8.STL" />
       </geometry>
     </collision>
@@ -572,33 +571,97 @@
       upper="0.05"
       effort="3"
-      velocity="5" />
-  </joint>
-  <!-- controller -->
-  <xacro:macro name="transmission_block" params="tran_name joint_name motor_name">
-    <transmission name="${tran_name}">
-        <type>transmission_interface/SimpleTransmission</type>
-        <joint name="${joint_name}">
-            <hardwareInterface>hardware_interface/PositionJointInterface</hardwareInterface>
-        </joint>
-        <actuator name="$motor_name">
-            <hardwareInterface>hardware_interface/PositionJointInterface</hardwareInterface>
-            <mechanicalReduction>1</mechanicalReduction>
-        </actuator>
-    </transmission>
-  </xacro:macro>
-  <xacro:transmission_block tran_name="tran1" joint_name="joint1" motor_name="joint1_motor"/>
-  <xacro:transmission_block tran_name="tran2" joint_name="joint2" motor_name="joint2_motor"/>
-  <xacro:transmission_block tran_name="tran3" joint_name="joint3" motor_name="joint3_motor"/>
-  <xacro:transmission_block tran_name="tran4" joint_name="joint4" motor_name="joint4_motor"/>
-  <xacro:transmission_block tran_name="tran5" joint_name="joint5" motor_name="joint5_motor"/>
-  <xacro:transmission_block tran_name="tran6" joint_name="joint6" motor_name="joint6_motor"/>
-  <xacro:transmission_block tran_name="tran7" joint_name="joint7" motor_name="joint7_motor"/>
-  <xacro:transmission_block tran_name="tran8" joint_name="joint8" motor_name="joint8_motor"/>
-  <!-- gazebo -->
-  <gazebo>
-    <plugin name="gazebo_ros_control" filename="libgazebo_ros_control.so">
-        <robotNamespace>/gazebo</robotNamespace>
-        <legacyModeNS>true</legacyModeNS>
-    </plugin>
-  </gazebo>
+      velocity="0" />
+  </joint>
+  <ros2_control name="GazeboSystem" type="system">
+    <hardware>
+        <plugin>gazebo_ros2_control/GazeboSystem</plugin>
+    </hardware>
+    <joint name="joint1">
+        <command_interface name="position">
+            <param name="min">-1</param>
+            <param name="max">1</param>
+        </command_interface>
+        <state_interface name="position">
+            <param name="initial_value">0.0</param>
+        </state_interface>
+        <state_interface name="velocity"/>
+    </joint>
+    <joint name="joint2">
+        <command_interface name="position">
+            <param name="min">-1</param>
+            <param name="max">1</param>
+        </command_interface>
+        <state_interface name="position">
+            <param name="initial_value">0.0</param>
+        </state_interface>
+        <state_interface name="velocity"/>
+    </joint>
+    <joint name="joint3">
+        <command_interface name="position">
+            <param name="min">-1</param>
+            <param name="max">1</param>
+        </command_interface>
+        <state_interface name="position">
+            <param name="initial_value">0.0</param>
+        </state_interface>
+        <state_interface name="velocity"/>
+    </joint>
+    <joint name="joint4">
+        <command_interface name="position">
+            <param name="min">-1</param>
+            <param name="max">1</param>
+        </command_interface>
+        <state_interface name="position">
+            <param name="initial_value">0.1</param>
+        </state_interface>
+        <state_interface name="velocity"/>
+    </joint>
+    <joint name="joint5">
+        <command_interface name="position">
+            <param name="min">-1</param>
+            <param name="max">1</param>
+        </command_interface>
+        <state_interface name="position">
+            <param name="initial_value">0.0</param>
+        </state_interface>
+        <state_interface name="velocity"/>
+    </joint>
+    <joint name="joint6">
+        <command_interface name="position">
+            <param name="min">-1</param>
+            <param name="max">1</param>
+        </command_interface>
+        <state_interface name="position">
+            <param name="initial_value">0.0</param>
+        </state_interface>
+        <state_interface name="velocity"/>
+    </joint>
+    <joint name="joint7">
+        <command_interface name="position">
+            <param name="min">-1</param>
+            <param name="max">1</param>
+        </command_interface>
+        <state_interface name="position">
+            <param name="initial_value">0.0</param>
+        </state_interface>
+        <state_interface name="velocity"/>
+    </joint>
+    <joint name="joint8">
+        <command_interface name="position">
+            <param name="min">-1</param>
+            <param name="max">1</param>
+        </command_interface>
+        <state_interface name="position">
+            <param name="initial_value">0.0</param>
+        </state_interface>
+        <state_interface name="velocity"/>
+    </joint>
+</ros2_control>
+<!-- gazebo -->
+<gazebo>
+  <plugin name="gazebo_ros2_control" filename="libgazebo_ros2_control.so">
+      <parameters> $(find y1_gazebo)/config/y1_with_gripper_controllers.yaml </parameters>
+      <robot_param_node>robot_state_publisher</robot_param_node>
+  </plugin>
+</gazebo>
 </robot>
