Commit message: fix urdf.

File: src/y1_controller/urdf/y10824_ee.urdf (robot description, URDF)
Before this commit: robot y1, 9 links, 8 joints
Links:
- link Link6: mass  0.479 ->  0.650

Commit message: add new launch

File: src/y1_controller/urdf/y10824_ee.urdf (robot description, URDF)
Before this commit: robot y1, 9 links, 8 joints
Links:
- link Link6: mass  0.479 ->  0.650
Joints:
- joint JOINT1: limit lower=-3.0 upper=3.0 effort=30 velocity=5 -> lower=-3.0 upper=3.0 effort=30 velocity=10
- joint JOINT2: limit lower=-3.5 upper=0.2 effort=100 velocity=5 -> lower=-3.5 upper=0.2 effort=120 velocity=10
- joint JOINT3: limit lower=-0.2 upper=4.1 effort=30 velocity=5 -> lower=-0.2 upper=3.5 effort=30 velocity=10
- joint JOINT4: limit lower=-2.5 upper=1.7 effort=10 velocity=20 -> lower=-2.5 upper=1.7 effort=30 velocity=10
- joint JOINT5: limit lower=-2.0 upper=2.0 effort=10 velocity=20 -> lower=-2.0 upper=2.0 effort=20 velocity=30
- joint JOINT6: limit lower=-3.0 upper=3.0 effort=10 velocity=20 -> lower=-3.0 upper=3.0 effort=20 velocity=30

Commit message: fix urdf y1_0824_ee

File: src/y1_controller/urdf/y10824_ee.urdf (robot description, URDF)
Before this commit: robot y1, 9 links, 8 joints
Joints:
- joint JOINT1: origin xyz=0 0 0 rpy=0 0 0 -> xyz=0 0 0.06675 rpy=0 0 0
- joint fixed_base_joint: axis 0 0 1 -> (none); origin xyz=0 0 0.06675 rpy=0 0 0 -> (none)

File: src/y1_controller/urdf/y1_no_gripper_0914.urdf (robot description, URDF)
Before this commit: robot y1, 8 links, 7 joints
Links:
- link Link1: geometry collision mesh filename=package://y1_description/meshes_y1/Link1.STL; visual mesh filename=package://y1_description/meshes_y1/Link1.STL
- link Link2: geometry collision mesh filename=package://y1_description/meshes_y1/Link2.STL; visual mesh filename=package://y1_description/meshes_y1/Link2.STL
- link Link3: geometry collision mesh filename=package://y1_description/meshes_y1/Link3.STL; visual mesh filename=package://y1_description/meshes_y1/Link3.STL
- link Link4: geometry collision mesh filename=package://y1_description/meshes_y1/Link4.STL; visual mesh filename=package://y1_description/meshes_y1/Link4.STL
- link Link5: geometry collision mesh filename=package://y1_description/meshes_y1/Link5.STL; visual mesh filename=package://y1_description/meshes_y1/Link5.STL
- link Link6: geometry collision mesh filename=package://y1_description/meshes_y1/Link6.STL; visual mesh filename=package://y1_description/meshes_y1/Link6.STL
- link base_link: geometry collision mesh filename=package://y1_description/meshes_y1/base_link.STL; visual mesh filename=package://y1_description/meshes_y1/base_link.STL

File: src/y1_controller/urdf/y1_with_gripper_2to1_0914.urdf (robot description, URDF)
Before this commit: robot y1, 9 links, 8 joints
Links:
- link Link1: geometry collision mesh filename=package://y1_description/meshes_y1/Link1.STL; visual mesh filename=package://y1_description/meshes_y1/Link1.STL
- link Link2: geometry collision mesh filename=package://y1_description/meshes_y1/Link2.STL; visual mesh filename=package://y1_description/meshes_y1/Link2.STL
- link Link3: geometry collision mesh filename=package://y1_description/meshes_y1/Link3.STL; visual mesh filename=package://y1_description/meshes_y1/Link3.STL
- link Link4: geometry collision mesh filename=package://y1_description/meshes_y1/Link4.STL; visual mesh filename=package://y1_description/meshes_y1/Link4.STL
- link Link5: geometry collision mesh filename=package://y1_description/meshes_y1/Link5.STL; visual mesh filename=package://y1_description/meshes_y1/Link5.STL
- link Link6: geometry collision mesh filename=package://y1_description/meshes_y1/Link6.STL; visual mesh filename=package://y1_description/meshes_y1/Link6.STL
- link base_link: geometry collision mesh filename=package://y1_description/meshes_y1/base_link.STL; visual mesh filename=package://y1_description/meshes_y1/base_link.STL
