Commit message: fix:modify urdf for rviz and kdl_solver.

File: src/y1_controller/urdf/y1_no_gripper.urdf (robot description, URDF)
Before this commit: robot y1, 8 links, 7 joints
Links:
- link Link1: geometry collision mesh filename=package://y1_description/meshes/Link1.STL; visual mesh filename=package://y1_description/meshes/Link1.STL
- link Link2: geometry collision mesh filename=package://y1_description/meshes/Link2.STL; visual mesh filename=package://y1_description/meshes/Link2.STL
- link Link3: mass 0.84000 -> 0.838; geometry collision mesh filename=package://y1_description/meshes/Link3.STL; visual mesh filename=package://y1_description/meshes/Link3.STL
- link Link4: geometry collision mesh filename=package://y1_description/meshes/Link4.STL; visual mesh filename=package://y1_description/meshes/Link4.STL
- link Link5: geometry collision mesh filename=package://y1_description/meshes/Link5.STL; visual mesh filename=package://y1_description/meshes/Link5.STL
- link Link6: mass 0.016469 -> 0.150000; geometry collision mesh filename=package://y1_description/meshes_y1/Link6.STL; visual mesh filename=package://y1_description/meshes_y1/Link6.STL
- link base_link: geometry collision mesh filename=package://y1_description/meshes/base_link.STL; visual mesh filename=package://y1_description/meshes/base_link.STL
Joints:
- joint JOINT6: axis 0 0 1 -> 1 0 0; origin xyz=0.0235 0 0.044 rpy=3.1416 1.5708 3.1416 -> xyz=0.0235 0 0.0440000000000001 rpy=-3.14159265330655 0 0

File: src/y1_controller/urdf/y1_with_gripper.urdf (robot description, URDF)
Before this commit: robot y1, 10 links, 9 joints
Links:
- removed link Claw_Link_L
- removed link Claw_Link_R
- link Link6: mass  0.479 -> 0.667000
Joints:
- removed joint Claw_Link_L
- removed joint Claw_Link_R
- joint JOINT1: limit lower=-3.0 upper=3.0 effort=30 velocity=5 -> lower=-3.0 upper=3.0 effort=30 velocity=10; origin xyz=0 0 0 rpy=0 0 0 -> xyz=0 0 0.06675 rpy=0 0 0
- joint JOINT2: limit lower=-3.5 upper=0.2 effort=100 velocity=5 -> lower=-3.5 upper=0.2 effort=120 velocity=10
- joint JOINT3: limit lower=-0.2 upper=4.1 effort=30 velocity=5 -> lower=-0.2 upper=3.5 effort=30 velocity=10
- joint JOINT4: limit lower=-2.5 upper=1.7 effort=10 velocity=20 -> lower=-2.5 upper=1.7 effort=30 velocity=10
- joint JOINT5: limit lower=-2.0 upper=2.0 effort=10 velocity=20 -> lower=-2.0 upper=2.0 effort=20 velocity=30
- joint JOINT6: axis 0 0 1 -> 1 0 0; limit lower=-3.0 upper=3.0 effort=10 velocity=20 -> lower=-3.0 upper=3.0 effort=20 velocity=30; origin xyz=0.0235 0 0.044 rpy=3.1416 1.5708 3.1416 -> xyz=0.0235 0 0.0440000000000001 rpy=-3.14159265330655 0 0
- joint fixed_base_joint: axis 0 0 1 -> (none); origin xyz=0 0 0.06675 rpy=0 0 0 -> (none)

File: src/y1_description/urdf/y1_no_gripper.urdf (robot description, URDF)
Before this commit: robot y1, 9 links, 8 joints
Links:
- removed link gripper_ee
- link Link1: mass 0.893000 -> 0.465086237348566
- link Link2: mass 1.028000 -> 1.00848298846255
- link Link3: mass 0.838 -> 0.839664047451371
- link Link4: mass 0.444000 -> 0.455192806560725
- link Link5: mass 0.363000 -> 0.373508569742983
- link Link6: mass  0.650 -> 0.0724468602058996
- link base_link: mass 0.632 -> 0.630484112037129
Joints:
- removed joint JOINT1
- removed joint JOINT2
- removed joint JOINT3
- removed joint JOINT4
- removed joint JOINT5
- removed joint JOINT6
- removed joint Link6_to_gripper_ee
- added joint Joint1: type revolute, parent base_link, child Link1, origin xyz=0 0 0.06675 rpy=0 0 0, axis 0 0 1, limit lower=-2.79 upper=2.79 effort=30 velocity=5
- added joint Joint2: type revolute, parent Link1, child Link2, origin xyz=0.00075 0 0.055 rpy=1.5707963267949 0 0, axis 0 0 1, limit lower=-3.14 upper=0 effort=100 velocity=5
- added joint Joint3: type revolute, parent Link2, child Link3, origin xyz=-0.28 0 0 rpy=0 0 0, axis 0 0 1, limit lower=0 upper=3.14 effort=30 velocity=5
- added joint Joint4: type revolute, parent Link3, child Link4, origin xyz=0.215000000000004 0.0630000000000073 0 rpy=0 0 0, axis 0 0 1, limit lower=-2.145 upper=1.413 effort=10 velocity=20
- added joint Joint5: type revolute, parent Link4, child Link5, origin xyz=0.0799999999999998 0.0519999999999981 0.000249997832942123 rpy=1.5707963267949 0 0, axis 0 0 1, limit lower=-1.482 upper=1.482 effort=10 velocity=20
- added joint Joint6: type revolute, parent Link5, child Link6, origin xyz=0.0235 0 0.0440000000000001 rpy=-3.14159265330655 0 0, axis 1 0 0, limit lower=-2.529 upper=2.529 effort=10 velocity=20
- joint fixed_base_joint: axis (none) -> 0 0 1; origin (none) -> xyz=0 0 0 rpy=0 0 0

File: src/y1_description/urdf/y1_with_gripper.urdf (robot description, URDF)
Before this commit: robot y1, 10 links, 9 joints
Links:
- added link gripper_base, mass 0.436099620967633; collision mesh filename=package://y1_description/meshes/gripper_base.STL; visual mesh filename=package://y1_description/meshes/gripper_base.STL
- link Claw_Link_L: mass 0.086 -> 0.0661690926183051
- link Claw_Link_R: mass 0.086 -> 0.0661690929217921
- link Link1: mass 0.893000 -> 0.465086237348566
- link Link2: mass 1.028000 -> 1.00848298846255
- link Link3: mass 0.838 -> 0.839664047451371
- link Link4: mass 0.444000 -> 0.455192806560725
- link Link5: mass 0.363000 -> 0.373508569742983
- link Link6: mass  0.479 -> 0.0724468602058996
- link base_link: mass 0.632 -> 0.630484112037129
Joints:
- removed joint JOINT1
- removed joint JOINT2
- removed joint JOINT3
- removed joint JOINT4
- removed joint JOINT5
- removed joint JOINT6
- added joint Joint1: type revolute, parent base_link, child Link1, origin xyz=0 0 0.06675 rpy=0 0 0, axis 0 0 1, limit lower=-2.79 upper=2.79 effort=30 velocity=5
- added joint Joint2: type revolute, parent Link1, child Link2, origin xyz=0.00075 0 0.055 rpy=1.5707963267949 0 0, axis 0 0 1, limit lower=-3.14 upper=0 effort=100 velocity=5
- added joint Joint3: type revolute, parent Link2, child Link3, origin xyz=-0.28 0 0 rpy=0 0 0, axis 0 0 1, limit lower=0 upper=3.14 effort=30 velocity=5
- added joint Joint4: type revolute, parent Link3, child Link4, origin xyz=0.215000000000004 0.0630000000000073 0 rpy=0 0 0, axis 0 0 1, limit lower=-2.145 upper=1.413 effort=10 velocity=20
- added joint Joint5: type revolute, parent Link4, child Link5, origin xyz=0.0799999999999998 0.0519999999999981 0.000249997832942123 rpy=1.5707963267949 0 0, axis 0 0 1, limit lower=-1.482 upper=1.482 effort=10 velocity=20
- added joint Joint6: type revolute, parent Link5, child Link6, origin xyz=0.0235 0 0.0440000000000001 rpy=-3.14159265330655 0 0, axis 1 0 0, limit lower=-2.529 upper=2.529 effort=10 velocity=20
- added joint gripper_base: type fixed, parent Link6, child gripper_base, origin xyz=0.0758 0 0 rpy=1.57079745225378 -1.57079631189374 1.57079520133601, axis 0 0 0
- joint Claw_Link_L: axis 0 0 -1 -> 1 0 0; limit lower=0 upper=0.045 effort=10 velocity=20 -> lower=-0.047 upper=0 effort=3 velocity=0; origin xyz=-0.0012063 -0.077001 0.07579 rpy=0 -1.5708 -1.5708 -> xyz=0 -0.00275000000000102 0 rpy=0 0 -1.5707963267949; parent Link6 -> gripper_base
- joint Claw_Link_R: axis 0 0 -1 -> 1 0 0; limit lower=0 upper=0.045 effort=10 velocity=20 -> lower=0 upper=0.047 effort=3 velocity=0; origin xyz=-0.0012063 0.076999 0.075791 rpy=0 -1.5708 -1.5708 -> xyz=0 0.00274999999999902 0 rpy=0 0 -1.5707963267949; parent Link6 -> gripper_base
- joint fixed_base_joint: origin xyz=0 0 0.06675 rpy=0 0 0 -> xyz=0 0 0 rpy=0 0 0

Commit message: fix end pose with urdf

File: src/y1_controller/urdf/y1_no_gripper.urdf (robot description, URDF)
Before this commit: robot y1, 8 links, 7 joints
Joints:
- joint JOINT1: axis 0 0 -1 -> 0 0 1
- joint JOINT3: limit lower=-0.2 upper=3.5 effort=30 velocity=10 -> lower=-0.2 upper=3.25 effort=30 velocity=10
- joint JOINT4: limit lower=-2.5 upper=1.7 effort=30 velocity=10 -> lower=-2.35 upper=1.6 effort=30 velocity=10
- joint JOINT5: limit lower=-2.0 upper=2.0 effort=20 velocity=30 -> lower=-1.6 upper=1.6 effort=20 velocity=30
- joint JOINT6: limit lower=-3.0 upper=3.0 effort=20 velocity=30 -> lower=-2.75 upper=2.75 effort=20 velocity=30

File: src/y1_controller/urdf/y1_with_gripper.urdf (robot description, URDF)
Before this commit: robot y1, 8 links, 7 joints
Joints:
- joint JOINT1: axis 0 0 -1 -> 0 0 1
- joint JOINT3: limit lower=-0.2 upper=3.5 effort=30 velocity=10 -> lower=-0.2 upper=3.25 effort=30 velocity=10
- joint JOINT4: limit lower=-2.5 upper=1.7 effort=30 velocity=10 -> lower=-2.35 upper=1.6 effort=30 velocity=10
- joint JOINT5: limit lower=-2.0 upper=2.0 effort=20 velocity=30 -> lower=-1.6 upper=1.6 effort=20 velocity=30
- joint JOINT6: limit lower=-3.0 upper=3.0 effort=20 velocity=30 -> lower=-2.75 upper=2.75 effort=20 velocity=30
